Commit message: Pugin Update Rate Changed

File: autonomous_car_description/urdf/autonomous_car_physical.xacro (robot description, xacro)
@@ -43,12 +43,12 @@
 </xacro:macro>
 <xacro:macro name="chassis_geometry">
-    <origin xyz="0 0 ${chassis_thickness/4}" rpy="0 0 0" />
+    <origin xyz="0 0 ${chassis_thickness/2}" rpy="0 0 0" />
     <geometry>
-        <box size="${chassis_width} ${chassis_length} ${chassis_thickness/2}"/>
+        <box size="${chassis_width} ${chassis_length} ${chassis_thickness}"/>
     </geometry>
 </xacro:macro>
 <xacro:macro name="chassis_inertial">
-    <origin xyz="0 0 ${chassis_thickness/4}" rpy="0 0 0" />
-    <xacro:box_inertial mass="${chassis_weight}" length="${chassis_length}" width="${chassis_width}" height="${chassis_thickness/2}" />
+    <origin xyz="0 0 ${chassis_thickness/8}" rpy="0 0 0" />
+    <xacro:box_inertial mass="${chassis_weight}" length="${chassis_length}" width="${chassis_width}" height="${chassis_thickness/4}" />
 </xacro:macro>
 <!-- Hinge -->

Commit message: Encoder is added

File: autonomous_car_description/urdf/autonomous_car_physical.xacro (robot description, xacro)
@@ -1,4 +1,5 @@
 <?xml version="1.0"?>
 <robot name="autonomous_car" xmlns:xacro="http://www.ros.org/wiki/xacro">
+<xacro:property name="pi" value="3.1415" />
 <!-- Chassis related properties -->
 <xacro:property name="chassis_width" value="1.100" />

Commit message: New Model is added

File: autonomous_car_description/urdf/autonomous_car_physical.xacro (robot description, xacro)
@@ -38,8 +38,8 @@
 <!-- Chassis -->
 <xacro:macro name="chassis_visual">
-    <origin xyz="0 0 ${chassis_thickness/2}" rpy="0 0 0" />
+    <origin xyz="0 -1.2 -0.08" rpy="${pi/2} 0 0" />
     <geometry>
-        <box size="${chassis_width} ${chassis_length} ${chassis_thickness}"/>
-    </geometry>
+        <mesh filename="package://autonomous_car_description/meshes/59RK.stl" scale="0.001 0.001 0.001"/>
+	</geometry>
 </xacro:macro>
 <xacro:macro name="chassis_geometry">
